File: hardware/BREAD_Slice.kicad_pcb (KiCad board)
At the start: 2 copper layers, 70 x 100 mm, 16 parts, among them J1 Conn_01x10_Female, U1 AP63205

Commit message: finalized pcb
Parts:
- added C10: 0.47u, Capacitor_SMD:C_0805_2012Metric_Pad1.18x1.45mm_HandSolder, B.Cu at (155.7, 59.8)
- added C11: 0.1u, Capacitor_SMD:C_0805_2012Metric_Pad1.18x1.45mm_HandSolder, B.Cu at (167.2, 98.3)
- added C12: 68n, Capacitor_SMD:C_0805_2012Metric_Pad1.18x1.45mm_HandSolder, B.Cu at (164.2, 93.6)
- added C13: 0.47u, Capacitor_SMD:C_0805_2012Metric_Pad1.18x1.45mm_HandSolder, B.Cu at (163.1, 90.5)
- added C14: 68n, Capacitor_SMD:C_0805_2012Metric_Pad1.18x1.45mm_HandSolder, B.Cu at (174.0, 90.8)
- added C15: 0.1u, Capacitor_SMD:C_0805_2012Metric_Pad1.18x1.45mm_HandSolder, B.Cu at (172.1, 84.7)
- added C16: 0.47u, Capacitor_SMD:C_0805_2012Metric_Pad1.18x1.45mm_HandSolder, B.Cu at (175.2, 83.9)
- added C5: 0.1u, Capacitor_SMD:C_0805_2012Metric_Pad1.18x1.45mm_HandSolder, B.Cu at (148.6, 74.0)
- added C6: 15n, Capacitor_SMD:C_0805_2012Metric_Pad1.18x1.45mm_HandSolder, B.Cu at (145.5, 69.3)
- added C7: 0.47u, Capacitor_SMD:C_0805_2012Metric_Pad1.18x1.45mm_HandSolder, B.Cu at (144.5, 66.3)
- added C8: 15n, Capacitor_SMD:C_0805_2012Metric_Pad1.18x1.45mm_HandSolder, B.Cu at (155.2, 65.8)
- added C9: 0.1u, Capacitor_SMD:C_0805_2012Metric_Pad1.18x1.45mm_HandSolder, B.Cu at (152.4, 60.9)
- added J2: Screw_Terminal_01x02, TerminalBlock_4Ucon:TerminalBlock_4Ucon_1x02_P3.50mm_Horizontal, F.Cu at (188.6, 67.5)
- added J3: SJ-3524-SMT, kml-custom:CUI_SJ-3524-SMT, F.Cu at (186.2, 101.5)
- added JP1: SolderJumper_3_Open, Jumper:SolderJumper-3_P2.0mm_Open_TrianglePad1.0x1.5mm, B.Cu at (179.7, 92.4)
- added JP2: SolderJumper_3_Open, Jumper:SolderJumper-3_P2.0mm_Open_TrianglePad1.0x1.5mm, B.Cu at (184.2, 90.7)
- added R1: 100k, Resistor_SMD:R_0805_2012Metric_Pad1.20x1.40mm_HandSolder, B.Cu at (143.4, 69.3)
- added R10: 24.9k, Resistor_SMD:R_1206_3216Metric_Pad1.30x1.75mm_HandSolder, F.Cu at (178.7, 67.5)
- added R11: 24.9k, Resistor_SMD:R_1206_3216Metric_Pad1.30x1.75mm_HandSolder, F.Cu at (182.1, 67.4)
- added R12: 24.9k, Resistor_SMD:R_1206_3216Metric_Pad1.30x1.75mm_HandSolder, F.Cu at (182.1, 72.8)
- added R13: 24.9k, Resistor_SMD:R_1206_3216Metric_Pad1.30x1.75mm_HandSolder, F.Cu at (186.0, 74.8)
- added R14: 22k, Resistor_SMD:R_0805_2012Metric_Pad1.20x1.40mm_HandSolder, B.Cu at (162.2, 93.6)
- added R15: 10k, Resistor_SMD:R_0805_2012Metric_Pad1.20x1.40mm_HandSolder, B.Cu at (164.2, 97.4)
- added R16: 10k, Resistor_SMD:R_0805_2012Metric_Pad1.20x1.40mm_HandSolder, B.Cu at (162.2, 97.4)
- added R17: 10k, Resistor_SMD:R_0805_2012Metric_Pad1.20x1.40mm_HandSolder, B.Cu at (167.0, 90.5)
- added R18: 10k, Resistor_SMD:R_0805_2012Metric_Pad1.20x1.40mm_HandSolder, B.Cu at (174.1, 97.1)
- added R19: 10k, Resistor_SMD:R_0805_2012Metric_Pad1.20x1.40mm_HandSolder, B.Cu at (175.0, 94.0)
- added R2: 10k, Resistor_SMD:R_0805_2012Metric_Pad1.20x1.40mm_HandSolder, B.Cu at (145.5, 73.2)
- added R20: 22k, Resistor_SMD:R_0805_2012Metric_Pad1.20x1.40mm_HandSolder, B.Cu at (170.9, 90.5)
- added R21: 10k, Resistor_SMD:R_0805_2012Metric_Pad1.20x1.40mm_HandSolder, B.Cu at (174.2, 86.9)
- added R3: 10k, Resistor_SMD:R_0805_2012Metric_Pad1.20x1.40mm_HandSolder, B.Cu at (143.5, 73.2)
- added R4: 10k, Resistor_SMD:R_0805_2012Metric_Pad1.20x1.40mm_HandSolder, B.Cu at (148.4, 66.1)
- added R5: 10k, Resistor_SMD:R_0805_2012Metric_Pad1.20x1.40mm_HandSolder, B.Cu at (156.1, 71.8)
- added R6: 10k, Resistor_SMD:R_0805_2012Metric_Pad1.20x1.40mm_HandSolder, B.Cu at (156.1, 69.0)
- added R7: 100k, Resistor_SMD:R_0805_2012Metric_Pad1.20x1.40mm_HandSolder, B.Cu at (152.2, 66.1)
- added R8: 10k, Resistor_SMD:R_0805_2012Metric_Pad1.20x1.40mm_HandSolder, B.Cu at (155.6, 62.3)
- added R9: 24.9k, Resistor_SMD:R_1206_3216Metric_Pad1.30x1.75mm_HandSolder, F.Cu at (178.6, 72.8)
- added RB1: 100, Resistor_SMD:R_0805_2012Metric_Pad1.20x1.40mm_HandSolder, B.Cu at (160.2, 65.5)
- added RB2: 100, Resistor_SMD:R_0805_2012Metric_Pad1.20x1.40mm_HandSolder, B.Cu at (178.5, 84.8)
- added TR1: ZMPT101, Transformer_THT:Transformer_Zeming_ZMPT101K, F.Cu at (171.0, 74.1)
- added TR2: ZMCT103C, Transformer_THT:Transformer_Zeming_ZMCT103C, F.Cu at (188.8, 90.7)
- added U2: LM358BIDR, Package_SO:SOIC-8_3.9x4.9mm_P1.27mm, B.Cu at (150.4, 70.1)
- added U3: MCP4161-104E/SN, Package_SO:SOIC-8_3.9x4.9mm_P1.27mm, B.Cu at (146.6, 62.1)
- added U4: LM358BIDR, Package_SO:SOIC-8_3.9x4.9mm_P1.27mm, B.Cu at (169.0, 94.4)
- added U5: MCP4161-104E/SN, Package_SO:SOIC-8_3.9x4.9mm_P1.27mm, B.Cu at (167.0, 86.5)
- J1: value Conn_01x10_Female -> Conn_01x10_Socket
- U1: footprint Package_TO_SOT_SMD:TSOT-23-6 -> kml-custom:SOIC_05WU-7_DIO
Connections:
- A1 pad 10: unconnected-(A1-D7-Pad10) -> /CS1
- A1 pad 11: unconnected-(A1-D8-Pad11) -> /CS2
- A1 pad 14: unconnected-(A1-D11-Pad14) -> /MOSI
- A1 pad 16: unconnected-(A1-D13-Pad16) -> /SCK
- A1 pad 19: /CURR1 -> /VOLT1
- A1 pad 20: /CURR2 -> unconnected-(A1-A1-Pad20)
- A1 pad 21: unconnected-(A1-A2-Pad21) -> /CURR1
Routing:
- net /SCK: track 0.00 -> 107.2 mm
- net /MOSI: track 0.00 -> 97.6 mm
- net +5V: track 104.2 -> 197.6 mm, vias 1 -> 10
- net /VOLT1: track 0.00 -> 70.9 mm, vias 0 -> 2
- net /CS1: track 0.00 -> 64.6 mm, vias 0 -> 2
- net /CS2: track 0.00 -> 46.7 mm, vias 0 -> 1
- net /CURR1: track 0.00 -> 40.8 mm
- net Net-(C10-Pad1): track 0.00 -> 21.5 mm
- net /Isolated AC Voltage Sensor1/AC_N: track 0.00 -> 20.8 mm
- net /Non-Invasive AC Current Sensor1/BIAS_1: track 0.00 -> 20.3 mm
- net /Isolated AC Voltage Sensor1/BIAS_1: track 0.00 -> 16.2 mm
- net GND: track 16.8 -> 32.8 mm, vias 20 -> 57
- net /Non-Invasive AC Current Sensor1/DIG_POT_A: track 0.00 -> 14.7 mm, vias 0 -> 2
- net /Isolated AC Voltage Sensor1/DIG_POT_A: track 0.00 -> 13.1 mm, vias 0 -> 2
- net Net-(U2A--): track 0.00 -> 12.4 mm
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- added copper zone on F.Cu, net GND
Other:
- board text added: "AC Current"
- board text added: "AC Voltage"
- board text added: "Ext. Jack"
- board text added: "LINE"
- board text added: "LINE RESISTORS"
- board text added: "NEUTRAL"
- board text added: "THT CT"
