File: hardware/BREAD_Slice.kicad_sch (KiCad schematic)
At the start: 17 parts, among them J1 Conn_01x10_Female, J4 Screw_Terminal_01x02, J5 Screw_Terminal_01x02, U1 AP63205

Commit message: finalized pcb
Parts:
- removed J1: Conn_01x10_Female, Connector_PinSocket_2.54mm:PinSocket_1x10_P2.54mm_Horizontal, symbol Connector:Conn_01x10_Female
- removed J4: Screw_Terminal_01x02, CRx:Pheonix Conn Term TDPT 4 2-SP-6,35-ZB, symbol Connector:Screw_Terminal_01x02
- added J1: Conn_01x10_Socket, Connector_PinSocket_2.54mm:PinSocket_1x10_P2.54mm_Horizontal, symbol Connector:Conn_01x10_Socket
- J2: renamed from J5; footprint CRx:Pheonix Conn Term TDPT 4 2-SP-6,35-ZB -> TerminalBlock_4Ucon:TerminalBlock_4Ucon_1x02_P3.50mm_Horizontal
- U1: footprint Package_TO_SOT_SMD:TSOT-23-6 -> kml-custom:SOIC_05WU-7_DIO; symbol SparkFun-DiscreteSemi:AP63205 -> kml-custom:AP63205WU-7
Connections:
- net Isolated AC Voltage Sensor2/AC_L is gone; now on net Isolated AC Voltage Sensor1/AC_N: J2.1 (Pin_1)
- net Isolated AC Voltage Sensor2/AC_N is gone; now on net Isolated AC Voltage Sensor1/AC_L: J2.2 (Pin_2)
- net +12V: now also J1.2 (Pin_2), J1.9 (Pin_9)
- net CURR1: now also A1.21 (A2); no longer A1.19 (A0)
- net ESTOP: now also J1.6 (Pin_6)
- net GNDPWR: now also J1.1 (Pin_1), J1.10 (Pin_10), J1.5 (Pin_5)
- net I2C_CLK: now also J1.3 (Pin_3)
- net I2C_DAT: now also J1.4 (Pin_4)
- net INT: now also J1.7 (Pin_7)
- net SYNC: now also J1.8 (Pin_8)
- net VOLT1: now also A1.19 (A0); no longer A1.21 (A2)
- net CS3: no longer names the net of A1.12 (D9)
- net CS4: no longer names the net of A1.13 (D10)
- net CURR2: no longer names the net of A1.20 (A1)
- net VOLT2: no longer names the net of A1.22 (A3)
- no-connect marks 12 -> 16
Other:
- removed sheet Isolated AC Voltage Sensor2
- removed sheet Non-Invasive AC Current Sensor2
- note added: "HAS SPACE FOR x2 OF EACH ONCE TESTED"
